Commit message: voglio piangere

File: ros2_iiwa/iiwa_description/urdf/camera.xacro (robot description, xacro)
@@ -5,5 +5,5 @@
       <parent link="${parent}"/>
       <child link="camera_link"/>
-      <origin xyz="0.02 0.0 0.0" rpy="0.0 -1.57 -3.14"/>
+      <origin xyz="0.02 0.0 0.0" rpy="0 0 0"/>
     </joint>
     <link name="camera_link">
@@ -17,4 +17,10 @@
       </visual>
     </link>
+    <joint name="camera_optical_joint" type="fixed">
+      <parent link="camera_link"/>
+      <child link="camera_link_optical"/>
+      <origin xyz="0.0 0.0 0.0" rpy="${-pi/2} 0 ${-pi/2}"/>
+    </joint>
+    <link name="camera_link_optical"></link>
     <gazebo>
       <plugin filename="gz-sim-sensors-system"
@@ -25,4 +31,5 @@
     <gazebo reference="camera_link">
       <sensor name="camera" type="camera">
+      <pose> 0 0 0 0 0 0 </pose>
         <camera>
           <horizontal_fov>1.047</horizontal_fov>

File: ros2_iiwa/iiwa_description/urdf/iiwa.urdf.xacro (robot description, xacro)
@@ -220,5 +220,5 @@
   </joint>
   <joint name="${prefix}joint_a7-tool0" type="fixed">
-      <origin rpy="0 0 0" xyz="0 0 0.154"/>
+      <origin rpy="3.14 -1.57 0" xyz="0 0 0.154"/>
       <parent link="${prefix}link_7"/>
       <child link="${prefix}tool0"/>
